Commit message: - Split minimal DIL-like UDS server from scenario UDS simulation - Add tracked target messages and TargetManager node - Route MissionExecutor and RViz visualization through /mission/tracked_targets - Keep /dil/frame as fallback input - Add simulation and live robot launch profiles - Improve fake Nav2 realism, robot visualization, odometry, TF, and wheel joints - Configure conservative target association for dense barn scenarios - Document launch/test workflow and current mission architecture

File: src/high_level_mission_planer/urdf/poultry_robot_visual.urdf (robot description, URDF)
Before this commit: robot poultry_robot_visual, 8 links, 7 joints
Joints:
- joint base_to_chassis: origin xyz=0 0 0 rpy=0 0 0 -> xyz=0 0 0.0907 rpy=0 0 0
- joint livox_joint: origin xyz=0.11 0.0 0.11 rpy=0.0 0.38 0.0 -> xyz=0.11 0.0 0.2007 rpy=0.0 0.38 0.0
- joint livox_mount_joint: origin xyz=0.11 0.0 0.078 rpy=0 0 0 -> xyz=0.11 0.0 0.1687 rpy=0 0 0
